Commit message: [Mini Quadrotor][Gazebo] add LiDAR sensor plugin to simualte Livox MID360

File: robots/mini_quadrotor/urdf/robot.urdf.xacro (robot description, xacro)
@@ -162,4 +162,14 @@
     </inertial>
   </xacro:extra_module>
+  <xacro:extra_module name = "livox_link" parent = "main_body" visible = "0" >
+    <origin xyz="0 0 ${0.0425 + 0.047}" rpy="0 0 0"/>
+    <inertial>
+      <mass value = "0" />
+      <origin xyz="0 0 0" rpy="0 0 0"/>
+      <inertia
+          ixx="0.0" ixy="0.0" ixz="0.0"
+          iyy="0.0" iyz="0.0" izz="0.0"/>
+    </inertial>
+  </xacro:extra_module>
   <!-- battery -->
   <xacro:extra_module name = "battery" parent = "main_body" visible = "1" model_url = "package://mini_quadrotor/urdf/mesh/turnigy_3S_2200mAh.dae" >
