Commit message: [Beetle]Modify the valve.urdf and beetle.urdf

File: robots/ninja/urdf/beetle.urdf.xacro (robot description, xacro)
@@ -58,78 +58,4 @@
       <origin rpy="0 0 0" xyz="0 0 0.12947"/>
       <axis xyz="0 0 1"/>
-    </joint>
-<!-- adding a manipulation link -->
-    <!-- <link name="manipulator_link_1">
-      <inertial>
-        <origin xyz="0.0071144 0.22 0.290" rpy="0 0 0"/>
-        <mass value="0.06"/>
-        <inertia
-            ixx="0.0001" iyy="0.0001" izz="0.0001"
-            ixy="0" ixz="0" iyz="0"/>
-      </inertial>
-      <visual>
-        <origin xyz="0.0071144 0.22 0.290" rpy="0 0 3.141592"/>
-        <geometry>
-          <mesh filename="package://beetle/urdf/mesh/Beetle_manipulator_v1.1.2.dae"/>
-        </geometry>
-      </visual>
-      <collision>
-        <origin xyz="0.0071144 0.22 0.290" rpy="0 0 0"/>
-        <geometry>
-          <box size="0.016 0.016 0.52"/>
-        </geometry>
-      </collision>
-    </link> -->
-     <link name="manipulator_link_1">
-      <inertial>
-        <origin xyz="-0.18 0.19 0.4" rpy="0 0 0"/>
-        <mass value="0.06"/>
-        <inertia
-            ixx="0.0001" iyy="0.0001" izz="0.0001"
-            ixy="0" ixz="0" iyz="0"/>
-      </inertial>
-      <visual>
-        <origin xyz="-0.18 0.19 0.2" rpy="0 0 3.141592"/>
-        <geometry>
-          <mesh filename="package://beetle/urdf/mesh/manipulator_v1.1.2.dae"/>
-        </geometry>
-      </visual>
-      <collision>
-        <origin xyz="-0.18 0.19 0.2" rpy="0 0 0"/>
-        <geometry>
-          <box size="0.016 0.016 0.52"/>
-        </geometry>
-      </collision>
-    </link>
-    <joint name="manipulator_joint_1" type="fixed">
-      <parent link="base_link"/>
-      <child link="manipulator_link_1"/>
-      <origin xyz="-0.18 0.19 0.2" rpy="0 0 0"/>
-    </joint>
-     <link name="manipulator_link_2">
-      <inertial>
-        <origin xyz="0.003 -0.18 0.3" rpy="0 0 0"/>
-        <mass value="0.06"/>
-        <inertia
-            ixx="0.0001" iyy="0.0001" izz="0.0001"
-            ixy="0" ixz="0" iyz="0"/>
-      </inertial>
-      <visual>
-        <origin xyz="0.003 -0.18 0.3" rpy="0 0 3.141592"/>
-        <geometry>
-          <mesh filename="package://beetle/urdf/mesh/manipulator_v1.1.2.dae"/>
-        </geometry>
-      </visual>
-      <collision>
-        <origin xyz="0.003 -0.18 0.3" rpy="0 0 0"/>
-        <geometry>
-          <box size="0.016 0.016 0.52"/>
-        </geometry>
-      </collision>
-    </link>
-    <joint name="manipulator_joint_2" type="fixed">
-      <parent link="base_link"/>
-      <child link="manipulator_link_2"/>
-      <origin xyz="0.003 -0.18 0.3" rpy="0 0 0"/>
     </joint>
     ## rotor arm macro
@@ -226,14 +152,4 @@
     </link>
     <xacro:damping_factor link="thrust${self}"/>
-## manipulation link (virtual)
-    <!-- <link name="manipulator_link_1_${self}">
-      <inertial>
-        <origin xyz="0 0 0" rpy="0 0 0"/>
-        <mass value="0.06"/>
-        <inertia
-            ixx="0.000001" iyy="0.000001" izz="0.000001"
-            ixy="0" ixz="0" iyz="0"/>
-      </inertial>
-    </link> -->
     #### joints ####
     #### gimbal joints ####
@@ -271,10 +187,4 @@
       <axis xyz="0 0 ${rotor_direction}"/>
     </joint>
-    #### manipulator joint (virtual) ####
-    <!-- <joint name="manipulator_joint_1_${self}" type="fixed">
-      <parent link="base_link"/>
-      <child link="manipulator_link_1"/>
-      <origin xyz="0.0071144 0.22 0.290" rpy="0 0 0"/>
-    </joint> -->
     <transmission name="rotor_tran${self}">
       <type>transmission_interface/SimpleTransmission</type>
