Commit message: [Beetle]Modify the Beetle.urdf.xacro

File: robots/beetle/urdf/beetle.urdf.xacro (robot description, xacro)
@@ -59,4 +59,26 @@
       <axis xyz="0 0 1"/>
     </joint>
+<!-- adding a manipulation link -->
+    <link name="manipulator_link${self}">
+      <inertial>
+        <origin xyz="0.0071144 0.22 0.290" rpy="0 0 0"/>
+        <mass value="0.06"/>
+        <inertia
+            ixx="0.0001" iyy="0.0001" izz="0.0001"
+            ixy="0" ixz="0" iyz="0"/>
+      </inertial>
+      <visual>
+        <origin xyz="0.0071144 0.22 0.290" rpy="0 0 3.141592"/>
+        <geometry>
+          <mesh filename="package://beetle/urdf/mesh/Beetle_manipulator_v1.1.2.dae"/>
+        </geometry>
+      </visual>
+      <collision>
+        <origin xyz="0.0071144 0.22 0.290" rpy="0 0 0"/>
+        <geometry>
+          <box size="0.016 0.016 0.52"/>
+        </geometry>
+      </collision>
+    </link>
     ## rotor arm macro
     <xacro:macro name="dummy_rotor_arm" params="id x y z yaw">
@@ -152,4 +174,14 @@
     </link>
     <xacro:damping_factor link="thrust${self}"/>
+## manipulation link (virtual)
+    <link name="manipulator_link${self}">
+      <inertial>
+        <origin xyz="0 0 0" rpy="0 0 0"/>
+        <mass value="0.06"/>
+        <inertia
+            ixx="0.000001" iyy="0.000001" izz="0.000001"
+            ixy="0" ixz="0" iyz="0"/>
+      </inertial>
+    </link>
     #### joints ####
     #### gimbal joints ####
@@ -187,4 +219,10 @@
       <axis xyz="0 0 ${rotor_direction}"/>
     </joint>
+    #### manipulator joint (virtual) ####
+    <joint name="manipulator_joint${self}" type="fixed">
+      <parent link="base_link"/>
+      <child link="manipulator_link"/>
+      <origin xyz="0.0071144 0.22 0.290" rpy="0 0 0"/>
+    </joint>
     <transmission name="rotor_tran${self}">
       <type>transmission_interface/SimpleTransmission</type>

Commit message: [Beetle]Build the simulation environment in gazebo with a upward vlve and beetle with manipulator

File: robots/beetle/urdf/beetle.urdf.xacro (robot description, xacro)
@@ -83,5 +83,5 @@
      <link name="manipulator_link_1">
       <inertial>
-        <origin xyz="-0.18 0.19 0.4" rpy="0 0 0"/>
+        <origin xyz="-0.18 0.19 -0.02" rpy="0 0 0"/>
         <mass value="0.06"/>
         <inertia
@@ -90,5 +90,5 @@
       </inertial>
       <visual>
-        <origin xyz="-0.18 0.19 0.2" rpy="0 0 3.141592"/>
+        <origin xyz="-0.18 0.19 -0.02" rpy="0 0 3.141592"/>
         <geometry>
           <mesh filename="package://beetle/urdf/mesh/manipulator_v1.1.2.dae"/>
@@ -96,7 +96,7 @@
       </visual>
       <collision>
-        <origin xyz="-0.18 0.19 0.2" rpy="0 0 0"/>
-        <geometry>
-          <box size="0.016 0.016 0.52"/>
+        <origin xyz="-0.18 0.19 -0.02" rpy="0 0 0"/>
+        <geometry>
+          <box size="0.016 0.016 0.42"/>
         </geometry>
       </collision>
@@ -105,9 +105,9 @@
       <parent link="base_link"/>
       <child link="manipulator_link_1"/>
-      <origin xyz="-0.18 0.19 0.2" rpy="0 0 0"/>
+      <origin xyz="-0.18 0.19 -0.02" rpy="0 0 0"/>
     </joint>
      <link name="manipulator_link_2">
       <inertial>
-        <origin xyz="0.003 -0.18 0.3" rpy="0 0 0"/>
+        <origin xyz="-0.18 -0.031 -0.02" rpy="0 0 0"/>
         <mass value="0.06"/>
         <inertia
@@ -116,5 +116,5 @@
       </inertial>
       <visual>
-        <origin xyz="0.003 -0.18 0.3" rpy="0 0 3.141592"/>
+        <origin xyz="-0.18 -0.031 -0.02" rpy="0 0 3.141592"/>
         <geometry>
           <mesh filename="package://beetle/urdf/mesh/manipulator_v1.1.2.dae"/>
@@ -122,7 +122,7 @@
       </visual>
       <collision>
-        <origin xyz="0.003 -0.18 0.3" rpy="0 0 0"/>
-        <geometry>
-          <box size="0.016 0.016 0.52"/>
+        <origin xyz="-0.18 -0.031 -0.02" rpy="0 0 0"/>
+        <geometry>
+          <box size="0.016 0.016 0.42"/>
         </geometry>
       </collision>
@@ -131,5 +131,5 @@
       <parent link="base_link"/>
       <child link="manipulator_link_2"/>
-      <origin xyz="0.003 -0.18 0.3" rpy="0 0 0"/>
+      <origin xyz="-0.18 -0.031 -0.02" rpy="0 0 0"/>
     </joint>
     ## rotor arm macro

File: robots/beetle/urdf/valve.urdf (robot description, URDF)
Before this commit: robot valve, 1 links, 5 joints
Links:
- added link i_beam, mass ${i_beam_mass}; collision box size=${i_beam_length} ${i_beam_width} ${i_beam_height}; visual box size=${i_beam_length} ${i_beam_width} ${i_beam_height}
Joints:
- added joint valve_to_i_beam_joint: type fixed, parent handle, child i_beam, origin xyz=0 0 ${valve_height - i_beam_height / 2 - 0.262} rpy=0 0 0, axis 0 0 1

Commit message: [Betle]Fixed the collison bug in gazebo

File: robots/beetle/urdf/beetle.urdf.xacro (robot description, xacro)
@@ -60,7 +60,7 @@
     </joint>
 <!-- adding a manipulation link -->
-    <!-- <link name="manipulator_link_1">
-      <inertial>
-        <origin xyz="0.0071144 0.22 0.290" rpy="0 0 0"/>
+     <link name="manipulator_link_1">
+      <inertial>
+        <origin xyz="-0.18 0.19 -0.02" rpy="0 0 0"/>
         <mass value="0.06"/>
         <inertia
@@ -69,19 +69,24 @@
       </inertial>
       <visual>
-        <origin xyz="0.0071144 0.22 0.290" rpy="0 0 3.141592"/>
-        <geometry>
-          <mesh filename="package://beetle/urdf/mesh/Beetle_manipulator_v1.1.2.dae"/>
-        </geometry>
-      </visual>
-      <collision>
-        <origin xyz="0.0071144 0.22 0.290" rpy="0 0 0"/>
-        <geometry>
-          <box size="0.016 0.016 0.52"/>
-        </geometry>
-      </collision>
-    </link> -->
-     <link name="manipulator_link_1">
-      <inertial>
-        <origin xyz="-0.18 0.19 -0.02" rpy="0 0 0"/>
+        <origin xyz="-0.18 0.19 -0.02" rpy="0 0 3.141592"/>
+        <geometry>
+          <mesh filename="package://beetle/urdf/mesh/manipulator_v1.1.2.dae"/>
+        </geometry>
+      </visual>
+      <collision>
+        <origin xyz="0.18 0.026 0.019" rpy="0 0 0"/>
+        <geometry>
+          <box size="0.016 0.016 0.5"/>
+        </geometry>
+      </collision>
+    </link>
+    <joint name="manipulator_joint_1" type="fixed">
+      <parent link="base_link"/>
+      <child link="manipulator_link_1"/>
+      <origin xyz="-0.18 0.19 -0.02" rpy="0 0 0"/>
+    </joint>
+     <link name="manipulator_link_2">
+      <inertial>
+        <origin xyz="-0.18 -0.031 -0.02" rpy="0 0 0"/>
         <mass value="0.06"/>
         <inertia
@@ -90,5 +95,5 @@
       </inertial>
       <visual>
-        <origin xyz="-0.18 0.19 -0.02" rpy="0 0 3.141592"/>
+        <origin xyz="-0.18 -0.031 -0.02" rpy="0 0 3.141592"/>
         <geometry>
           <mesh filename="package://beetle/urdf/mesh/manipulator_v1.1.2.dae"/>
@@ -96,33 +101,7 @@
       </visual>
       <collision>
-        <origin xyz="-0.18 0.19 -0.02" rpy="0 0 0"/>
-        <geometry>
-          <box size="0.016 0.016 0.42"/>
-        </geometry>
-      </collision>
-    </link>
-    <joint name="manipulator_joint_1" type="fixed">
-      <parent link="base_link"/>
-      <child link="manipulator_link_1"/>
-      <origin xyz="-0.18 0.19 -0.02" rpy="0 0 0"/>
-    </joint>
-     <link name="manipulator_link_2">
-      <inertial>
-        <origin xyz="-0.18 -0.031 -0.02" rpy="0 0 0"/>
-        <mass value="0.06"/>
-        <inertia
-            ixx="0.0001" iyy="0.0001" izz="0.0001"
-            ixy="0" ixz="0" iyz="0"/>
-      </inertial>
-      <visual>
-        <origin xyz="-0.18 -0.031 -0.02" rpy="0 0 3.141592"/>
-        <geometry>
-          <mesh filename="package://beetle/urdf/mesh/manipulator_v1.1.2.dae"/>
-        </geometry>
-      </visual>
-      <collision>
-        <origin xyz="-0.18 -0.031 -0.02" rpy="0 0 0"/>
-        <geometry>
-          <box size="0.016 0.016 0.42"/>
+        <origin xyz="0.18 -0.196 0.019" rpy="0 0 0"/>
+        <geometry>
+          <box size="0.016 0.016 0.5"/>
         </geometry>
       </collision>
